Commit message: Tried to add multi-robot compatibility...fail

File: movee_description/urdf/gazebo_plugins.xacro (robot description, xacro)
@@ -4,5 +4,5 @@
   <gazebo>
     <plugin name="gazebo_ros_control" filename="libgazebo_ros_control.so">
-       <robotNamespace>${robot_namespace}</robotNamespace>
+       <!-- <robotNamespace>${robot_namespace}</robotNamespace> -->
        <robotSimType>gazebo_ros_control/DefaultRobotHWSim</robotSimType>
     </plugin>
@@ -17,12 +17,12 @@
       <topic>__default_topic__</topic>
       <plugin filename="libgazebo_ros_imu_sensor.so" name="imu_plugin">
-        <topicName>imu</topicName>
+        <!-- <robotNamespace>${robot_namespace}</robotNamespace> -->
+        <topicName>/imu</topicName>
         <bodyName>imu_link</bodyName>
-        <robotNamespace>${robot_namespace}</robotNamespace>
         <updateRateHZ>10.0</updateRateHZ>
         <gaussianNoise>0.0</gaussianNoise>
         <xyzOffset>0 0 0</xyzOffset>
         <rpyOffset>0 0 0</rpyOffset>
-        <frameName>imu_link</frameName>
+        <frameName>/imu_link</frameName>
       </plugin>
       <pose>0 0 0 0 0 0</pose>
@@ -47,11 +47,11 @@
       </camera>
       <plugin name="camera_controller" filename="libgazebo_ros_camera.so">
+        <!-- <robotNamespace>${robot_namespace}</robotNamespace> -->
         <alwaysOn>true</alwaysOn>
         <updateRate>0.0</updateRate>
-        <cameraName>mybot/camera1</cameraName>
+        <cameraName>rrbot/camera1</cameraName>
         <imageTopicName>image_raw</imageTopicName>
         <cameraInfoTopicName>camera_info</cameraInfoTopicName>
-        <frameName>camera</frameName>
-        <robotNamespace>${robot_namespace}</robotNamespace>
+        <frameName>camera_link</frameName>
         <hackBaseline>0.07</hackBaseline>
         <distortionK1>0.0</distortionK1>
@@ -94,7 +94,7 @@
       </ray>
       <plugin name="gazebo_ros_head_hokuyo_controller" filename="libgazebo_ros_gpu_laser.so">
-        <topicName>/mybot/laser/scan</topicName>
-        <frameName>hokuyo</frameName>
-        <robotNamespace>${robot_namespace}</robotNamespace>
+        <!-- <robotNamespace>/robot12</robotNamespace> -->
+        <topicName>/laser/scan</topicName>
+        <frameName>hokuyo_link</frameName>
       </plugin>
     </sensor>
@@ -120,11 +120,11 @@
       <alwaysOn>true</alwaysOn>
       <updateRate>1.0</updateRate>
-      <robotNamespace>${robot_namespace}</robotNamespace>
+      <!-- <robotNamespace>${robot_namespace}</robotNamespace> -->
       <cameraName>${depth_camera_name}_ir</cameraName>
-      <imageTopicName>/${depth_camera_name}/color/image_raw</imageTopicName>
-      <cameraInfoTopicName>/${depth_camera_name}/color/camera_info</cameraInfoTopicName>
-      <depthImageTopicName>/${depth_camera_name}/depth/image_raw</depthImageTopicName>
-      <depthImageInfoTopicName>/${depth_camera_name}/depth/camera_info</depthImageInfoTopicName>
-      <pointCloudTopicName>/${depth_camera_name}/depth/points</pointCloudTopicName>
+      <imageTopicName>/color/image_raw</imageTopicName>
+      <cameraInfoTopicName>/color/camera_info</cameraInfoTopicName>
+      <depthImageTopicName>/depth/image_raw</depthImageTopicName>
+      <depthImageInfoTopicName>/depth/camera_info</depthImageInfoTopicName>
+      <pointCloudTopicName>/depth/points</pointCloudTopicName>
       <frameName>depth_sensor</frameName>
       <pointCloudCutoff>0.5</pointCloudCutoff>

File: movee_description/urdf/robot_parameters.xacro (robot description, xacro)
@@ -1,14 +1,14 @@
 <?xml version="1.0" ?>
 <robot xmlns:xacro="http://www.ros.org/wiki/xacro">
-  <xacro:arg name="training_wheels" default="true" />
-  <xacro:property name="wheel_mass" value="0.5" />
-  <xacro:property name="wheel_radius" value="0.1" />
-  <xacro:property name="wheel_thickness" value="0.05" />
-  <xacro:property name="wheelbase" value="0.5" />
-  <xacro:property name="thigh_length" value="0.4" />
-  <xacro:property name="thigh_conrod_length" value="0.5" />
-  <xacro:property name="calf_length" value="0.4" />
-  <xacro:property name="body_mass" value="10" />
-  <xacro:property name="robot_namespace" value="/" />
+  <xacro:arg name="training_wheels" default="false" />
+  <xacro:property name="wheel_mass" default="0.5" />
+  <xacro:property name="wheel_radius" default="0.1" />
+  <xacro:property name="wheel_thickness" default="0.05" />
+  <xacro:property name="wheelbase" default="0.5" />
+  <xacro:property name="thigh_length" default="0.4" />
+  <xacro:property name="thigh_conrod_length" default="0.5" />
+  <xacro:property name="calf_length" default="0.4" />
+  <xacro:property name="body_mass" default="10" />
+  <xacro:property name="robot_namespace" default="" />
   <xacro:property name="depth_camera_name" value="Creative"/>
   <xacro:property name="depth_camera_mass" value="0.1"/>
