Commit message: Added senors, reworked files but issue with the TFs (due to the /namespace in robot_parameters/xacro ?

File: movee_description/urdf/friction.xacro (robot description, xacro)
@@ -1,4 +1,4 @@
 <?xml version="1.0"?>
-<robot name="teeterbot_friction" xmlns:xacro="http://www.ros.org/wiki/xacro" >
+<robot xmlns:xacro="http://www.ros.org/wiki/xacro" >
   <gazebo reference="chassis_link" >
     <material>Gazebo/>Red</material>
@@ -16,3 +16,30 @@
     <mu2>0.5</mu2>
   </gazebo>
+  <gazebo reference="imu_link" >
+    <material>Gazebo/>Red</material>
+  </gazebo>
+  <gazebo reference="camera_link" >
+    <material>Gazebo/>ZincYellow</material>
+  </gazebo>
+  <gazebo reference="depth_sensor_link" >
+    <material>Gazebo/TurquoiseGlow></material>
+  </gazebo>
+  <gazebo reference="training_wheel_1">
+    <mu1>0.8</mu1>
+    <mu2>0.8</mu2>
+    <maxVel>0.0</maxVel>
+    <minDepth>0.001</minDepth>
+  </gazebo>
+  <gazebo reference="training_wheel_2">
+    <mu1>0.8</mu1>
+    <mu2>0.8</mu2>
+    <maxVel>0.0</maxVel>
+    <minDepth>0.001</minDepth>
+  </gazebo>
+  <gazebo reference="training_wheel_3">
+    <mu1>0.8</mu1>
+    <mu2>0.8</mu2>
+    <maxVel>0.0</maxVel>
+    <minDepth>0.001</minDepth>
+  </gazebo>
 </robot>

File: movee_description/urdf/movee.urdf (robot description, URDF)
Before this commit: robot Movee, 10 links, 9 joints
Joints:
- joint hip_pivot_conrod_left: limit lower=-3.14 upper=3.14 effort=-1.0 velocity=-1.0 -> lower=-3.14 upper=3.14 effort=-1.0 velocity=12
- joint hip_pivot_conrod_right: limit lower=-3.14 upper=3.14 effort=-1.0 velocity=-1.0 -> lower=-3.14 upper=3.14 effort=100 velocity=12
- joint hip_pivot_left: limit lower=0.4 upper=1 effort=-1.0 velocity=-1.0 -> lower=0.4 upper=1 effort=100 velocity=12
- joint hip_pivot_right: limit lower=0.4 upper=1 effort=-1.0 velocity=-1.0 -> lower=0.4 upper=1 effort=100 velocity=12
- joint knee_pivot_left: limit lower=0.1 upper=1 effort=-1.0 velocity=-1.0 -> lower=0.1 upper=1 effort=100 velocity=12
- joint knee_pivot_right: limit lower=0.1 upper=1 effort=-1.0 velocity=-1.0 -> lower=0.1 upper=1 effort=100 velocity=12

File: movee_description/urdf/robot_parameters.xacro (robot description, xacro)
@@ -1,9 +1,29 @@
 <?xml version="1.0" ?>
 <robot xmlns:xacro="http://www.ros.org/wiki/xacro">
-  <xacro:property name="link_00_name" value="base_link" />
-  <xacro:property name="link_01_name" value="link_01" />
-  <xacro:property name="link_02_name" value="link_02" />
-  <xacro:property name="link_03_name" value="link_03" />
-  <xacro:property name="link_04_name" value="link_04" />
-  <xacro:property name="link_05_name" value="link_05" />
+  <xacro:arg name="training_wheels" default="true" />
+  <xacro:property name="wheel_mass" value="0.5" />
+  <xacro:property name="wheel_radius" value="0.1" />
+  <xacro:property name="wheel_thickness" value="0.05" />
+  <xacro:property name="wheelbase" value="0.5" />
+  <xacro:property name="thigh_length" value="0.4" />
+  <xacro:property name="thigh_conrod_length" value="0.5" />
+  <xacro:property name="calf_length" value="0.4" />
+  <xacro:property name="body_mass" value="10" />
+  <xacro:property name="robot_namespace" value="/" />
+  <xacro:property name="depth_camera_name" value="Creative"/>
+  <xacro:property name="depth_camera_mass" value="0.1"/>
+  <!-- ###################################################MATERIAL DEFINITION######################################## -->
+<!-- ######################################################################################################### -->
+  <material name="red">
+    <color rgba="0.9 0.15 0.15 1.0"/>
+  </material>
+ <material name="green">
+    <color rgba="0.2 0.8 0.2 1.0"/>
+  </material>
+  <material name="orange">
+    <color rgba="0.64 0.313939 0.095351 1.0"/>
+  </material>
+   <material name="blue">
+    <color rgba="0.12 0.42 0.8 1.0"/>
+  </material>
 </robot>

Commit message: new telop launch and robot moving with bugs

File: movee_description/urdf/friction.xacro (robot description, xacro)
@@ -3,16 +3,29 @@
   <gazebo reference="chassis_link" >
     <material>Gazebo/>Red</material>
-    <mu1>0.0</mu1>
-    <mu2>0.0</mu2>
+        <friction>
+            <mu>0</mu>
+            <mu2>0</mu2>
+            <slip1>1.0</slip1>
+            <slip2>1.0</slip2>
+        </friction>
+  </gazebo>
+  <gazebo reference="base_link" >
+    <material>Gazebo/>Red</material>
+        <friction>
+            <mu>0</mu>
+            <mu2>0</mu2>
+            <slip1>1.0</slip1>
+            <slip2>1.0</slip2>
+        </friction>
   </gazebo>
   <gazebo reference="wheel_right" >
     <material>Gazebo/Grey</material>
-    <mu1>0.5</mu1>
-    <mu2>0.5</mu2>
+    <mu1>10000</mu1>
+    <mu2>10000</mu2>
   </gazebo>
   <gazebo reference="wheel_left" >
     <material>Gazebo/Grey</material>
-    <mu1>0.5</mu1>
-    <mu2>0.5</mu2>
+    <mu1>10000</mu1>
+    <mu2>10000</mu2>
   </gazebo>
   <gazebo reference="imu_link" >

File: movee_description/urdf/gazebo_plugins.xacro (robot description, xacro)
@@ -8,4 +8,23 @@
     </plugin>
   </gazebo>
+  <gazebo>
+    <plugin name="differential_drive_controller" filename="libgazebo_ros_diff_drive.so">
+      <legacyMode>false</legacyMode>
+      <alwaysOn>true</alwaysOn>
+      <updateRate>20</updateRate>
+      <leftJoint>wheel_pivot_left</leftJoint>
+      <rightJoint>wheel_pivot_right</rightJoint>
+      <wheelSeparation>0.5</wheelSeparation>
+      <wheelDiameter>0.2</wheelDiameter>
+      <torque>10</torque>
+      <commandTopic>cmd_vel</commandTopic>
+      <odometryTopic>odom</odometryTopic>
+      <odometryFrame>odom</odometryFrame>
+      <robotBaseFrame>chassis</robotBaseFrame>
+    </plugin>
+  </gazebo>
+  <gazebo reference="chassis">
+      <material>Gazebo/Orange</material>
+    </gazebo>
   <!-- imu -->
   <gazebo reference="imu_link">
@@ -67,5 +86,5 @@
     <sensor type="gpu_ray" name="head_hokuyo_sensor">
       <pose>0 0 0 0 0 0</pose>
-      <visualize>true</visualize>
+      <visualize>false</visualize>
       <update_rate>40</update_rate>
       <ray>
@@ -85,5 +104,6 @@
         <noise>
           <type>gaussian</type>
-          <!-- Noise parameters based on published spec for Hokuyo laser
+          <!-- Noise parameters
+ based on published spec for Hokuyo laser
                achieving "+-30mm" accuracy at range < 10m.  A mean of 0.0m and
                stddev of 0.01m will put 99.7% of samples within 0.03m of the true
